File: Hardware/SparkFun_Noisy_Cricket.sch (EAGLE design)
At the start: 27 parts, among them U1 LM4853

Commit message: Design Review Changes
- Moved JP1 further away from POT1
- Added JP2 to short C3 and increase bass frequency reponse in mono
operation
Parts:
- added JP2: JUMPER-SMT_2_NO_NO-SILK, SparkFun-Jumpers:JUMPER-SMT_2_NO_NO-SILK
- C1, C2: value 0.1uF -> 1.0uF; device SparkFun-Capacitors:0.1UF-0603-25V-5% -> SparkFun-Capacitors:1.0UF-0603-16V-10%
Connections:
- removed net N$8: C3.+, POT1G1.E, U1.LOUT
- new net LOUT+: C3.+, JP2.1, POT1G1.E, U1.LOUT
- net LOUT: now also JP2.2
Other:
- note added: "JP1 Note: - Open (Default): Stereo Output (Outputs: Left, Right, GND) - Closed: Mono Output (Outputs: Left, Mono) In mono mode, connect speaker to Left and Mono, NOT ground!"
- note added: "JP2 Note: - Jumper should be open when in stereo operation. - In mono operation, JP2 can be either opened or closed. - When closed, JP2 shorts C3, which will allow lower frequencies to pass more easily."
- note removed: "JP1 Note: - Open (Default): Stereo Output (Left, Right, GND) - Closed: Mono Output (Left, Mono) In mono mode, connect speaker to Left and Mono, NOT ground!"
- moved on the sheet: JP1, POT1G3
Changed lines of the file:
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@@
 <part name="FRAME1" library="SparkFun-Aesthetics" deviceset="FRAME-LETTER" device=""/>
 <part name="U1" library="SparkFun-IC-Amplifiers" deviceset="LM4853" device="" value="LM4853"/>
-<part name="C1" library="SparkFun-Capacitors" deviceset="0.1UF" device="-0603-25V-5%" value="0.1uF"/>
-<part name="C2" library="SparkFun-Capacitors" deviceset="0.1UF" device="-0603-25V-5%" value="0.1uF"/>
+<part name="C1" library="SparkFun-Capacitors" deviceset="1.0UF" device="-0603-16V-10%" value="1.0uF"/>
+<part name="C2" library="SparkFun-Capacitors" deviceset="1.0UF" device="-0603-16V-10%" value="1.0uF"/>
 <part name="R1" library="SparkFun-Resistors" deviceset="20KOHM" device="-0603-1/10W-1%" value="20k"/>
 <part name="R2" library="SparkFun-Resistors" deviceset="20KOHM" device="-0603-1/10W-1%" value="20k"/>
@@
 <part name="LOGO1" library="SparkFun-Aesthetics" deviceset="SFE_LOGO_NAME" device=".1_INCH"/>
 <part name="LOGO2" library="SparkFun-Aesthetics" deviceset="OSHW-LOGO" device="S"/>
+<part name="JP2" library="SparkFun-Jumpers" deviceset="JUMPER-SMT_2_NO" device="_NO-SILK" value=""/>
 </parts>
 <sheets>
 <sheet>
 <plain>
-<text x="150.622" y="47.498" size="1.778" layer="97">JP1 Note:
-- Open (Default): Stereo Output (Left, Right, GND)
-- Closed: Mono Output (Left, Mono)
-In mono mode, connect speaker to Left and Mono,
-NOT ground!</text>
-<wire x1="248.92" y1="78.74" x2="147.32" y2="78.74" width="0.2032" layer="97" style="shortdash"/>
-<wire x1="147.32" y1="78.74" x2="147.32" y2="35.56" width="0.2032" layer="97" style="shortdash"/>
-<wire x1="147.32" y1="78.74" x2="99.06" y2="78.74" width="0.2032" layer="97" style="shortdash"/>
+<text x="104.902" y="50.038" size="1.778" layer="97">JP1 Note:
+- Open (Default): Stereo Output
+ (Outputs: Left, Right, GND)
+- Closed: Mono Output
+ (Outputs: Left, Mono)
+In mono mode, connect speaker
+to Left and Mono, NOT ground!</text>
+<wire x1="248.92" y1="78.74" x2="99.06" y2="78.74" width="0.2032" layer="97" style="shortdash"/>
+<wire x1="99.06" y1="78.74" x2="99.06" y2="35.56" width="0.2032" layer="97" style="shortdash"/>
 <wire x1="99.06" y1="78.74" x2="99.06" y2="185.42" width="0.2032" layer="97" style="shortdash"/>
 <wire x1="99.06" y1="78.74" x2="0" y2="78.74" width="0.2032" layer="97" style="shortdash"/>
-<wire x1="147.32" y1="35.56" x2="0" y2="35.56" width="0.2032" layer="97" style="shortdash"/>
-<text x="149.86" y="73.66" size="2.54" layer="94">Jumper</text>
+<wire x1="99.06" y1="35.56" x2="0" y2="35.56" width="0.2032" layer="97" style="shortdash"/>
+<text x="101.6" y="73.66" size="2.54" layer="94">Jumper</text>
 <text x="101.6" y="180.34" size="2.54" layer="94">Audio Amplifier</text>
 <text x="2.54" y="180.34" size="2.54" layer="94">Header</text>
@@
 <text x="238.506" y="7.112" size="2.54" layer="94">v01</text>
 <text x="33.02" y="165.1" size="2.54" layer="97">VIN: 2.4 - 5.5V</text>
-<text x="53.34" y="43.18" size="1.778" layer="97">Switch Current: 3A MAX</text>
+<text x="10.16" y="45.72" size="1.778" layer="97">Switch Current: 3A MAX</text>
+<wire x1="99.06" y1="35.56" x2="147.32" y2="35.56" width="0.2032" layer="97" style="shortdash"/>
+<text x="170.18" y="48.26" size="1.778" layer="97">JP2 Note:
+- Jumper should be open when in stereo operation.
+- In mono operation, JP2 can be either opened or
+ closed.
+- When closed, JP2 shorts C3, which will allow
+ lower frequencies to pass more easily.</text>
 </plain>
 <instances>
@@
 <instance part="GND4" gate="1" x="167.64" y="93.98"/>
 <instance part="GND25" gate="1" x="124.46" y="93.98"/>
-<instance part="JP1" gate="G$1" x="228.6" y="58.42" rot="R90"/>
-<instance part="GND5" gate="1" x="228.6" y="48.26"/>
+<instance part="JP1" gate="G$1" x="162.56" y="60.96" rot="R90"/>
+<instance part="GND5" gate="1" x="162.56" y="50.8"/>
 <instance part="R7" gate="G$1" x="154.94" y="127" smashed="yes">
 <attribute name="NAME" x="154.94" y="125.476" size="1.778" layer="95" font="vector" rot="R180" align="bottom-center"/>
@@
 <instance part="SUPPLY1" gate="G$1" x="50.8" y="144.78"/>
 <instance part="SUPPLY4" gate="G$1" x="58.42" y="144.78"/>
-<instance part="POT1" gate="G3" x="68.58" y="50.8"/>
-<instance part="SUPPLY5" gate="G$1" x="60.96" y="55.88"/>
-<instance part="SUPPLY6" gate="G$1" x="76.2" y="55.88"/>
+<instance part="POT1" gate="G3" x="25.4" y="53.34" smashed="yes">
+<attribute name="NAME" x="25.4" y="54.864" size="1.778" layer="95" align="bottom-center"/>
+</instance>
+<instance part="SUPPLY5" gate="G$1" x="17.78" y="58.42"/>
+<instance part="SUPPLY6" gate="G$1" x="33.02" y="58.42"/>
 <instance part="C6" gate="G$1" x="218.44" y="154.94" rot="MR0"/>
 <instance part="GND7" gate="1" x="218.44" y="147.32"/>
@@
 <instance part="LOGO1" gate="G$1" x="20.32" y="7.62"/>
 <instance part="LOGO2" gate="G$1" x="116.84" y="17.78"/>
+<instance part="JP2" gate="G$1" x="208.28" y="68.58"/>
 </instances>
 <busses>
@@
 </segment>
 </net>
-<net name="N$8" class="0">
+<net name="LOUT+" class="0">
 <segment>
 <pinref part="U1" gate="G$1" pin="LOUT"/>
@@
 <wire x1="210.82" y1="106.68" x2="210.82" y2="132.08" width="0.1524" layer="91"/>
 <junction x="210.82" y="132.08"/>
+<label x="203.708" y="132.334" size="1.27" layer="95"/>
+</segment>
+<segment>
+<pinref part="JP2" gate="G$1" pin="1"/>
+<wire x1="203.2" y1="68.58" x2="200.66" y2="68.58" width="0.1524" layer="91"/>
+<label x="200.66" y="68.58" size="1.27" layer="95" rot="R180" xref="yes"/>
 </segment>
 </net>
@@
 <wire x1="48.26" y1="121.92" x2="53.34" y2="121.92" width="0.1524" layer="91"/>
 <label x="53.34" y="121.92" size="1.27" layer="95" xref="yes"/>
+</segment>
+<segment>
+<pinref part="JP2" gate="G$1" pin="2"/>
+<wire x1="213.36" y1="68.58" x2="215.9" y2="68.58" width="0.1524" layer="91"/>
+<label x="215.9" y="68.58" size="1.27" layer="95" xref="yes"/>
 </segment>
 </net>
@@
 <segment>
 <pinref part="POT1" gate="G3" pin="2"/>
-<wire x1="73.66" y1="50.8" x2="76.2" y2="50.8" width="0.1524" layer="91"/>
-<wire x1="76.2" y1="50.8" x2="76.2" y2="55.88" width="0.1524" layer="91"/>
+<wire x1="30.48" y1="53.34" x2="33.02" y2="53.34" width="0.1524" layer="91"/>
+<wire x1="33.02" y1="53.34" x2="33.02" y2="58.42" width="0.1524" layer="91"/>
 <pinref part="SUPPLY6" gate="G$1" pin="5V"/>
 </segment>
@@
 <segment>
 <pinref part="JP1" gate="G$1" pin="1"/>
-<wire x1="228.6" y1="53.34" x2="228.6" y2="50.8" width="0.1524" layer="91"/>
+<wire x1="162.56" y1="55.88" x2="162.56" y2="53.34" width="0.1524" layer="91"/>
 <pinref part="GND5" gate="1" pin="GND"/>
 </segment>
@@
 <segment>
 <pinref part="JP1" gate="G$1" pin="2"/>
-<wire x1="228.6" y1="63.5" x2="228.6" y2="66.04" width="0.1524" layer="91"/>
-<wire x1="228.6" y1="66.04" x2="226.06" y2="66.04" width="0.1524" layer="91"/>
-<label x="226.06" y="66.04" size="1.27" layer="95" rot="R180" xref="yes"/>
+<wire x1="162.56" y1="66.04" x2="162.56" y2="68.58" width="0.1524" layer="91"/>
+<wire x1="162.56" y1="68.58" x2="160.02" y2="68.58" width="0.1524" layer="91"/>
+<label x="160.02" y="68.58" size="1.27" layer="95" rot="R180" xref="yes"/>
 </segment>
 </net>
@@
 <segment>
 <pinref part="POT1" gate="G3" pin="1"/>
-<wire x1="63.5" y1="50.8" x2="60.96" y2="50.8" width="0.1524" layer="91"/>
-<wire x1="60.96" y1="50.8" x2="60.96" y2="55.88" width="0.1524" layer="91"/>
+<wire x1="20.32" y1="53.34" x2="17.78" y2="53.34" width="0.1524" layer="91"/>
+<wire x1="17.78" y1="53.34" x2="17.78" y2="58.42" width="0.1524" layer="91"/>
 <pinref part="SUPPLY5" gate="G$1" pin="VIN"/>
 </segment>

Commit message: v10 Changes
- Replaced C1/C2 with X7R capacitors with a better low end frequency
response.
- Moved C3/C4 further away from POT1.
- Replaced R1/R2 with 2.2k resistors instead of 20k.
- Added lines to top silk to separate Power/Input/Output sections.
- Changed "Mono Enable" silk on bottom layer to "Mono Output".
Parts:
- R1, R2: value 20k -> 2.2k; device SparkFun-Resistors:20KOHM-0603-1/10W-1% -> SparkFun-Resistors:2.2KOHM-0603-1/10W-1%
Changed lines of the file:
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@@
 <layer number="59" name="tCarbon" color="7" fill="1" visible="no" active="no"/>
 <layer number="60" name="bCarbon" color="7" fill="1" visible="no" active="no"/>
+<layer number="88" name="SimResults" color="9" fill="1" visible="yes" active="yes"/>
+<layer number="89" name="SimProbes" color="9" fill="1" visible="yes" active="yes"/>
 <layer number="90" name="Modules" color="5" fill="1" visible="yes" active="yes"/>
 <layer number="91" name="Nets" color="2" fill="1" visible="yes" active="yes"/>
@@
 <part name="C1" library="SparkFun-Capacitors" deviceset="1.0UF" device="-0603-16V-10%" value="1.0uF"/>
 <part name="C2" library="SparkFun-Capacitors" deviceset="1.0UF" device="-0603-16V-10%" value="1.0uF"/>
-<part name="R1" library="SparkFun-Resistors" deviceset="20KOHM" device="-0603-1/10W-1%" value="20k"/>
-<part name="R2" library="SparkFun-Resistors" deviceset="20KOHM" device="-0603-1/10W-1%" value="20k"/>
+<part name="R1" library="SparkFun-Resistors" deviceset="2.2KOHM" device="-0603-1/10W-1%" value="2.2k"/>
+<part name="R2" library="SparkFun-Resistors" deviceset="2.2KOHM" device="-0603-1/10W-1%" value="2.2k"/>
 <part name="C3" library="SparkFun-Capacitors" deviceset="100UF-POLAR" device="-25V-20%(ELEC)" value="100uF"/>
 <part name="C4" library="SparkFun-Capacitors" deviceset="100UF-POLAR" device="-25V-20%(ELEC)" value="100uF"/>

Commit message: v10 Changes cont.
- New 1.0uF capacitors weren't added to previous commit. Added correct
capacitors.
Parts:
- C1, C2, C5, C6: device SparkFun-Capacitors:1.0UF-0603-16V-10% -> SparkFun-Capacitors:1.0UF-0603-16V-10%-X7R
Changed lines of the file:
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@@
 <part name="FRAME1" library="SparkFun-Aesthetics" deviceset="FRAME-LETTER" device=""/>
 <part name="U1" library="SparkFun-IC-Amplifiers" deviceset="LM4853" device="" value="LM4853"/>
-<part name="C1" library="SparkFun-Capacitors" deviceset="1.0UF" device="-0603-16V-10%" value="1.0uF"/>
-<part name="C2" library="SparkFun-Capacitors" deviceset="1.0UF" device="-0603-16V-10%" value="1.0uF"/>
+<part name="C1" library="SparkFun-Capacitors" deviceset="1.0UF" device="-0603-16V-10%-X7R" value="1.0uF"/>
+<part name="C2" library="SparkFun-Capacitors" deviceset="1.0UF" device="-0603-16V-10%-X7R" value="1.0uF"/>
 <part name="R1" library="SparkFun-Resistors" deviceset="2.2KOHM" device="-0603-1/10W-1%" value="2.2k"/>
 <part name="R2" library="SparkFun-Resistors" deviceset="2.2KOHM" device="-0603-1/10W-1%" value="2.2k"/>
@@
 <part name="GND3" library="SparkFun-PowerSymbols" deviceset="GND" device=""/>
 <part name="POT1" library="SparkFun-Resistors" deviceset="POTENTIOMETER_DUAL_W/SWITCH" device="" value="20k"/>
-<part name="C5" library="SparkFun-Capacitors" deviceset="1.0UF" device="-0603-16V-10%" value="1.0uF"/>
+<part name="C5" library="SparkFun-Capacitors" deviceset="1.0UF" device="-0603-16V-10%-X7R" value="1.0uF"/>
 <part name="GND4" library="SparkFun-PowerSymbols" deviceset="GND" device=""/>
 <part name="GND25" library="SparkFun-PowerSymbols" deviceset="GND" device=""/>
@@
 <part name="SUPPLY5" library="SparkFun-PowerSymbols" deviceset="VIN" device=""/>
 <part name="SUPPLY6" library="SparkFun-PowerSymbols" deviceset="5V" device=""/>
-<part name="C6" library="SparkFun-Capacitors" deviceset="1.0UF" device="-0603-16V-10%" value="1.0uF"/>
+<part name="C6" library="SparkFun-Capacitors" deviceset="1.0UF" device="-0603-16V-10%-X7R" value="1.0uF"/>
 <part name="GND7" library="SparkFun-PowerSymbols" deviceset="GND" device=""/>
 <part name="SUPPLY7" library="SparkFun-PowerSymbols" deviceset="5V" device=""/>
