File: Production/SparkFun_Noisy_Cricket-Panel_V10.brd (EAGLE design)
At the start: 251.5 x 116.8 mm, 790 parts, among them U1 LM4853, U10 LM4853, U11 LM4853, U12 LM4853, U13 LM4853, U14 LM4853, U15 LM4853, U16 LM4853, U17 LM4853, U18 LM4853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

Commit message: moved to origin
Parts:
- moved POT14 9.70 mm to (134.4, 45.5)
- moved POT13 9.70 mm to (134.4, 19.6)
- moved C104 9.70 mm to (152.7, 52.6)
- moved C105 9.70 mm to (161.9, 36.7)
- moved C107 9.70 mm to (152.8, 45.5)
- moved C109 9.70 mm to (152.7, 80.0)
- moved C110 9.70 mm to (152.7, 78.5)
- moved C115 9.70 mm to (152.7, 105.9)
- moved C116 9.70 mm to (152.7, 104.4)
- moved C117 9.70 mm to (161.9, 88.5)
- moved C128 9.70 mm to (186.7, 52.6)
- moved C129 9.70 mm to (196.0, 36.7)
- moved C131 9.70 mm to (186.8, 45.5)
- moved C133 9.70 mm to (186.7, 80.0)
- moved C134 9.70 mm to (186.7, 78.5)
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Other:
- outline, holes or cut-outs redrawn
